File: EnviroHATv6/EnviroHAT.kicad_pcb (KiCad board)
At the start: 2 copper layers, 100 x 100 mm, 61 parts, among them J1 Conn_01x10_Pin, J2 Conn_01x32_Socket, J3 Conn_01x32_Socket, J4 MICROXNJ, Q1 AO3400A, Q2 AO3400A, Q4 PT42-21C/TR8, Q5 AO3400A, U2 FT234XD-R, U3 CAT24C256, U4 VCNL36821S, U5 MP2602DQ-LF-Z, U6 XC6206P332MR, U7 AMS1117-5.0

Commit message: Update to v 6.2
Parts:
- J2, J3: value Conn_01x32_Socket -> Conn_01x33_Socket; footprint Connector_PinSocket_2.54mm:PinSocket_1x32_P2.54mm_Vertical -> Connector_PinSocket_2.54mm:PinSocket_1x33_P2.54mm_Vertical
- moved R1 5.28 mm to (139.2, 95.6)
- moved R2 4.96 mm to (127.9, 92.5)
- moved R3 3.02 mm to (142.9, 102.5)
- moved R4 3.02 mm to (146.6, 102.5)
- moved R5 3.02 mm to (150.2, 102.5)
- moved J3 0.08 mm to (132.1, 48.0)
Connections:
- J2 pad 1: unconnected-(J2-Pin_1-Pad1) -> +3V3
- J2 pad 32: GND -> unconnected-(J2-Pin_32-Pad32)
- J3 pad 18: unconnected-(J3-Pin_18-Pad18) -> Sensor_SDA
- J3 pad 19: unconnected-(J3-Pin_19-Pad19) -> Sensor_SCL
- J3 pad 2: unconnected-(J3-Pin_2-Pad2) -> GND
- J3 pad 20: Sensor_SDA -> unconnected-(J3-Pin_20-Pad20)
- J3 pad 21: Sensor_SCL -> unconnected-(J3-Pin_21-Pad21)
- J3 pad 23: unconnected-(J3-Pin_23-Pad23) -> AOUT
- J3 pad 24: AOUT -> unconnected-(J3-Pin_24-Pad24)
- J3 pad 25: unconnected-(J3-Pin_25-Pad25) -> DIG_OUT
- J3 pad 26: DIG_OUT -> unconnected-(J3-Pin_26-Pad26)
- J3 pad 32: GND -> unconnected-(J3-Pin_32-Pad32)
Routing:
- net +3V3: track 254.0 -> 296.8 mm
- net GND: track 86.0 -> 98.7 mm, vias 5 -> 6
- net USB_Detect: track 143.8 -> 131.2 mm
- net Sensor_SCL: track 62.5 -> 71.0 mm
- net Sensor_SDA: track 61.6 -> 69.9 mm
- net AOUT: track 49.7 -> 55.5 mm
- net Net-(U4-SDA): track 52.6 -> 57.4 mm
- net /MCU Submodule/USART FTDI RXD: track 126.8 -> 130.6 mm
- net /Sensing Submodule/GPIO1: track 67.6 -> 71.1 mm
- net /MCU Submodule/USART FTDI TXD: track 115.9 -> 119.3 mm
- net Net-(U4-SCL): track 52.1 -> 55.1 mm
- net DIG_OUT: track 18.5 -> 20.8 mm
- net USBDP: track 75.1 -> 74.0 mm
- net Net-(U3-SCL): track 35.7 -> 36.7 mm
- net Net-(U3-SDA): track 28.3 -> 29.2 mm
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Other:
- board text added: "Group 15 V6.2"
- board text removed: "Group 15 V6.0"

Commit message: PCB Cleanup V6.3
Parts:
- removed J2, J3: Conn_01x33_Socket, Connector_PinSocket_2.54mm:PinSocket_1x33_P2.54mm_Vertical
- added U8: ~, footprints:STM32F051C6T6, F.Cu at (124.2, 75.0)
- BT1: footprint footprints:18650_HOLDER_TH -> footprints:18650_Holder_SMD
- moved U3 43.3 mm to (144.1, 116.1)
- moved U2 38.5 mm to (139.8, 88.5)
- moved R29 34.9 mm to (131.4, 116.1)
- moved R28 34.9 mm to (129.2, 116.1)
- moved R8 34.9 mm to (135.9, 116.2)
- moved R9 29.0 mm to (121.6, 100.5)
- moved R27 29.0 mm to (121.6, 102.8)
- moved R6 28.9 mm to (122.4, 92.5)
- moved D2 13.2 mm to (122.7, 134.4)
- moved D1 10.3 mm to (132.5, 134.1)
- moved Q1 10.3 mm to (132.5, 127.3)
- moved Q2 10.3 mm to (120.4, 125.6)
- moved R7 10.3 mm to (127.8, 133.6)
- moved BT1 2.11 mm to (177.3, 82.8)
Routing:
- net GND: track 98.7 -> 498.2 mm
- net Sensor_GPIO1: track 69.9 -> 34.2 mm, vias 1 -> 0
- net /MCU Submodule/USART FTDI RTS: track 18.6 -> 53.6 mm, vias 1 -> 2
- net USBDN: track 82.0 -> 52.4 mm, vias 0 -> 2
- net +BATT: track 116.5 -> 89.1 mm
- net /MCU Submodule/USART FTDI RXD: track 130.6 -> 103.5 mm, vias 1 -> 0
- net Net-(U3-SCL): track 36.7 -> 14.4 mm
- net Net-(D1-A): track 29.2 -> 7.51 mm
- net /MCU Submodule/USART FTDI CTS: track 12.0 -> 31.6 mm, vias 1 -> 3
- net +5V: track 99.8 -> 80.3 mm
- net Net-(D2-K): track 3.82 -> 23.2 mm
- net USBDP: track 74.0 -> 54.7 mm, vias 0 -> 2
- net AOUT: track 55.5 -> 72.2 mm, vias 1 -> 3
- net Sensor_SDA: track 69.9 -> 85.7 mm, vias 1 -> 2
- net /Sensing Submodule/GPIO1: track 71.1 -> 56.6 mm, vias 2 -> 3
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Other:
- board size 100 x 100 mm -> 75 x 100 mm
- board text added: "Group 15 V6.3"
- board text removed: "Group 15 V6.2"
