File: EnviroHATv6/Power Management Submodule.kicad_sch (KiCad schematic)
At the start: 32 parts, among them J4 MICROXNJ, U5 MP2602DQ-LF-Z, U6 XC6206P332MR, U7 AMS1117-5.0

Commit message: PCB Cleanup V6.3
Parts:
- BT1: footprint footprints:18650_HOLDER_TH -> footprints:18650_Holder_SMD; now left out of the parts list
Changed lines of the file:
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@@
   )
   (symbol (lib_id "Device:Battery") (at 106.68 137.16 0) (unit 1)
-    (in_bom yes) (on_board yes) (dnp no) (fields_autoplaced)
+    (in_bom no) (on_board yes) (dnp no) (fields_autoplaced)
     (property "Reference" "BT1" (at 110.49 136.144 0)
       (effects (font (size 1.27 1.27)) (justify left))
@@
       (effects (font (size 1.27 1.27)) (justify left))
     )
-    (property "Footprint" "footprints:18650_HOLDER_TH" (at 106.68 135.636 90)
+    (property "Footprint" "footprints:18650_Holder_SMD" (at 106.68 135.636 90)
       (effects (font (size 1.27 1.27)) hide)
     )
